Commit message: Updates to QBP URDF to include 4 casters as fixed supports. Modified visual elements and collision volumes to match external surface of QBot platform geometry

File: qbot_platform/urdf/qbot_platform.urdf (robot description, URDF)
Before this commit: robot qbot_platform, 3 links, 2 joints
Links:
- added link base_footprint
- added link downward_camera_link
- added link front_left_caster, mass 0.01; collision cylinder length=0.025 radius=0.045; visual cylinder length=0.025 radius=0.045
- added link front_right_caster, mass 0.005; collision cylinder length=0.025 radius=0.045; visual cylinder length=0.025 radius=0.045
- added link imu_link
- added link lidar_link
- added link realsense_depth_link
- added link realsense_rgb_link
- added link rear_left_caster, mass 0.005; collision cylinder length=0.025 radius=0.045; visual cylinder length=0.025 radius=0.045
- added link rear_right_caster, mass 0.005; collision cylinder length=0.025 radius=0.045; visual cylinder length=0.025 radius=0.045
- link base_link: geometry collision box size=0.3 0.01 0.18; collision box size=0.3 0.01 0.18
- link left_wheel: geometry collision cylinder length=0.025 radius=0.045; visual mesh filename=package://qbot_platform/meshes/qbot_platform_wheel.stl scale=0.001 0.001 0.001
- link right_wheel: geometry collision cylinder length=0.025 radius=0.045; visual mesh filename=package://qbot_platform/meshes/qbot_platform_wheel.stl scale=0.001 0.001 0.001
Joints:
- added joint base_link_joint: type fixed, parent base_footprint, child base_link, origin xyz=0 0 0.112 rpy=0 0 0
- added joint downward_camera_joint: type fixed, parent base_link, child downward_camera_link, origin xyz=0.03 0 -0.05 rpy=3.14159 0 -1.5708
- added joint front_left_caster_joint: type fixed, parent base_link, child front_left_caster, origin xyz=0.13 0.13 -0.06 rpy=-1.57 -1.57 0, axis 0 0 1
- added joint front_right_caster_joint: type fixed, parent base_link, child front_right_caster, origin xyz=0.13 -0.13 -0.06 rpy=-1.57 -1.57 0, axis 0 0 1
- added joint imu_joint: type fixed, parent base_link, child imu_link, origin xyz=0 0 -0.04 rpy=0 0 0
- added joint lidar_joint: type fixed, parent base_link, child lidar_link, origin xyz=0.221 0 0.1 rpy=0 0 0
- added joint realsense_depth_joint: type fixed, parent base_link, child realsense_depth_link, origin xyz=0.261 0 0.03 rpy=-1.5708 0 -1.5708
- added joint realsense_rgb_joint: type fixed, parent base_link, child realsense_rgb_link, origin xyz=0.261 0.033 0.03 rpy=-1.5708 0 -1.5708
- added joint rear_left_caster_joint: type fixed, parent base_link, child rear_left_caster, origin xyz=-0.13 0.13 -0.06 rpy=-1.57 -1.57 0, axis 0 0 1
- added joint rear_right_caster_joint: type fixed, parent base_link, child rear_right_caster, origin xyz=-0.13 -0.13 -0.06 rpy=-1.57 -1.57 0, axis 0 0 1
- joint left_wheel_joint: limit lower=-1e+16 upper=1e+16 effort=300 velocity=2 -> lower=-1e16 upper=1e16 effort=300 velocity=2; origin xyz=-0.015 0.1965 -0.06 rpy=1.57 1.57 0 -> xyz=0 0.1965 -0.0605 rpy=-1.57 -1.57 0
- joint right_wheel_joint: limit lower=-1e+16 upper=1e+16 effort=300 velocity=2 -> lower=-1e16 upper=1e16 effort=300 velocity=2; origin xyz=-0.015 -0.1965 -0.06 rpy=1.57 1.57 0 -> xyz=0.0 -0.1965 -0.0605 rpy=-1.57 -1.57 0
