Commit message: Modified QCar URDF and added QCar 2 URDF
Qcar URDF has modified collision volumes and has all sensors defined with the correct orientation for wheels and sensors. DAE mesh files have been deleted.
Qcar 2 URDF has been added with updated STL. Inertias and weights defined after testing with real device.

File: qcar2/urdf/QCar2.urdf (robot description, URDF)
Before this commit: robot QCar, 14 links, 13 joints
Links:
- removed link base
- removed link hubfl
- removed link hubfr
- removed link realsense
- removed link wheelfl
- removed link wheelfr
- removed link wheelrl
- removed link wheelrr
- added link base_link, mass 3.275; collision box size=.03 .15 .115; collision box size=.037 .15 .115
- added link hub_frontLeft, mass 0.1; visual mesh filename=package://qcar2/meshes/QCarSteeringHubL.stl scale=0.001 0.001 0.001
- added link hub_frontRight, mass 0.1; visual mesh filename=package://qcar2/meshes/QCarSteeringHubR.stl scale=0.001 0.001 0.001
- added link realsenseDepth
- added link realsenseRGB
- added link wheel_frontLeft, mass 0.1; collision cylinder length=0.025 radius=0.033; visual mesh filename=package://qcar2/meshes/QCarWheel.stl scale=0.001 0.001 0.001
- added link wheel_frontRight, mass 0.1; collision cylinder length=0.025 radius=0.033; visual mesh filename=package://qcar2/meshes/QCarWheel.stl scale=0.001 0.001 0.001
- added link wheel_rearLeft, mass 0.1; collision cylinder length=0.025 radius=0.033; visual mesh filename=package://qcar2/meshes/QCarWheel.stl scale=0.001 0.001 0.001
- added link wheel_rearRight, mass 0.1; collision cylinder length=0.025 radius=0.033; visual mesh filename=package://qcar2/meshes/QCarWheel.stl scale=0.001 0.001 0.001
- link lidar: mass 0.1 -> None; geometry visual mesh filename=package://qcar2/meshes/QCar2Lidar.stl scale=0.1 0.1 0.1
Joints:
- removed joint base_hubfl_joint
- removed joint base_hubfr_joint
- removed joint base_wheelrl_joint
- removed joint base_wheelrr_joint
- removed joint body_lidar_joint
- removed joint hubfl_wheelfl_joint
- removed joint hubfr_wheelfr_joint
- removed joint realsense_joint
- added joint hub_frontLeft_joint: type revolute, parent base_link, child hub_frontLeft, origin xyz=0.12960 0.05590 0.03338 rpy=0 0 0, axis 0 0 1, limit lower=-0.5236 upper=0.5236 effort=300 velocity=2
- added joint hub_frontRight_joint: type revolute, parent base_link, child hub_frontRight, origin xyz=0.12960 -0.05590 0.03338 rpy=0 0 0, axis 0 0 1, limit lower=-0.5236 upper=0.5236 effort=300 velocity=2
- added joint lidar_joint: type fixed, parent base_link, child lidar, origin xyz=-0.0139 0 .194 rpy=0 0 0, axis 0 0 1
- added joint realsenseDepth_joint: type fixed, parent base_link, child realsenseDepth, origin xyz=0.095 -0.003 0.176 rpy=-1.5708 0 -1.5708
- added joint realsenseRGB_joint: type fixed, parent base_link, child realsenseRGB, origin xyz=0.095 0.034 0.176 rpy=-1.5708 0 -1.5708
- added joint wheel_frontLeft_joint: type continuous, parent hub_frontLeft, child wheel_frontLeft, origin xyz=0 0 0 rpy=-1.5708 0 0, axis 0 0 1
- added joint wheel_frontRight_joint: type continuous, parent hub_frontRight, child wheel_frontRight, origin xyz=0 0 0 rpy=-1.5708 0 0, axis 0 0 1
- added joint wheel_rearLeft_joint: type continuous, parent base_link, child wheel_rearLeft, origin xyz=-0.12765 0.05610 0.03338 rpy=-1.5708 0 0, axis 0 0 1
- added joint wheel_rearRight_joint: type continuous, parent base_link, child wheel_rearRight, origin xyz=-0.12765 -0.05610 0.03338 rpy=-1.5708 0 0, axis 0 0 1
- joint csi_back_joint: origin xyz=-0.165 0 0.094 rpy=-1.5708 0 1.5708 -> xyz=-0.165 -0.0005 0.1095 rpy=-1.5708 0 1.5708; parent base -> base_link
- joint csi_front_joint: origin xyz=0.193 0 0.094 rpy=-1.5708 0 -1.5708 -> xyz=0.198 0 0.1095 rpy=-1.5708 0 -1.5708; parent base -> base_link
- joint csi_left_joint: origin xyz=0.0135 0.048 0.094 rpy=-1.5708 0 0 -> xyz=0.0155 0.051 0.1095 rpy=-1.5708 0 0; parent base -> base_link
- joint csi_right_joint: origin xyz=0.014 -0.0674 0.094 rpy=-1.5708 0 3.14159 -> xyz=0.0155 -0.072 0.1095 rpy=-1.5708 0 3.14159; parent base -> base_link
- joint imu_joint: origin xyz=0.127 0.0223 0.0895 rpy=0 0 0 -> xyz=0.0119 0 0.0896 rpy=0 0 0; parent base -> base_link

Commit message: Updated colors for QCar2 urdf. change name to lowercase to match qbot platform

File: qcar2/urdf/QCar2.urdf (robot description, URDF)
Before this commit: robot qcar2, 15 links, 14 joints
Links:
- link lidar: geometry visual cylinder length=0.0194 radius=0.04; visual mesh filename=package://qcar2/meshes/QCar2Lidar.stl scale=0.1 0.1 0.1
